Commit message: WIP working com

File: ros2_control/cubemars.ros2_control.xacro (robot description, xacro)
@@ -1,13 +1,13 @@
 <?xml version="1.0"?>
 <robot xmlns:xacro="http://www.ros.org/wiki/xacro">
-  <xacro:macro name="cubemars_ak" params="name prefix can_id Kp Kd vel_min vel_max effort_min effort_max pos_min:=-12.5 pos_max:=12.5 Kp_min:=0 Kp_max:=500 Kd_min:=0 Kd_max:=5">
+  <xacro:macro name="cubemars_ak" params="name prefix can_id kp kd vel_min vel_max effort_min effort_max pos_min:=-12.5 pos_max:=12.5 kp_min:=0 kp_max:=500 kd_min:=0 kd_max:=5">
     <joint name="${prefix}${name}">
       <param name="can_id">${can_id}</param>
-      <param name="Kp">${Kp}</param>
-      <param name="Kd">${Kd}</param>
-      <param name="Kp_min">${Kp_min}</param>
-      <param name="Kp_max">${Kp_max}</param>
-      <param name="Kd_min">${Kd_min}</param>
-      <param name="Kd_max">${Kd_max}</param>
+      <param name="kp">${kp}</param>
+      <param name="kd">${kd}</param>
+      <param name="kp_min">${kp_min}</param>
+      <param name="kp_max">${kp_max}</param>
+      <param name="kd_min">${kd_min}</param>
+      <param name="kd_max">${kd_max}</param>
       <command_interface name="position">
         <param name="min">${pos_min}</param>
@@ -28,22 +28,22 @@
     </joint>
   </xacro:macro>
-  <xacro:macro name="AK10-9" params="name prefix can_id Kp Kd">
-    <xacro:cubemars_ak name="${name}" prefix="${prefix}" can_id="${can_id}" Kp="${Kp}" Kd="${Kd}" vel_min="-50.0" vel_max="50.0" effort_min="-65.0" effort_max="65.0" />
+  <xacro:macro name="AK10-9" params="name prefix can_id kp kd">
+    <xacro:cubemars_ak name="${name}" prefix="${prefix}" can_id="${can_id}" kp="${kp}" kd="${kd}" vel_min="-50.0" vel_max="50.0" effort_min="-65.0" effort_max="65.0" />
   </xacro:macro>
-  <xacro:macro name="AK60-6" params="name prefix can_id Kp Kd">
-    <xacro:cubemars_ak name="${name}" prefix="${prefix}" can_id="${can_id}" Kp="${Kp}" Kd="${Kd}" vel_min="-45.0" vel_max="45.0" effort_min="-15.0" effort_max="15.0" />
+  <xacro:macro name="AK60-6" params="name prefix can_id kp kd">
+    <xacro:cubemars_ak name="${name}" prefix="${prefix}" can_id="${can_id}" kp="${kp}" kd="${kd}" vel_min="-45.0" vel_max="45.0" effort_min="-15.0" effort_max="15.0" />
   </xacro:macro>
-  <xacro:macro name="AK70-10" params="name prefix can_id Kp Kd">
-    <xacro:cubemars_ak name="${name}" prefix="${prefix}" can_id="${can_id}" Kp="${Kp}" Kd="${Kd}" vel_min="-50.0" vel_max="50.0" effort_min="-25.0" effort_max="25.0" />
+  <xacro:macro name="AK70-10" params="name prefix can_id kp kd">
+    <xacro:cubemars_ak name="${name}" prefix="${prefix}" can_id="${can_id}" kp="${kp}" kd="${kd}" vel_min="-50.0" vel_max="50.0" effort_min="-25.0" effort_max="25.0" />
   </xacro:macro>
-  <xacro:macro name="AK80-5" params="name prefix can_id Kp Kd">
-    <xacro:cubemars_ak name="${name}" prefix="${prefix}" can_id="${can_id}" Kp="${Kp}" Kd="${Kd}" vel_min="-76.0" vel_max="76.0" effort_min="-12.0" effort_max="12.0" />
+  <xacro:macro name="AK80-5" params="name prefix can_id kp kd">
+    <xacro:cubemars_ak name="${name}" prefix="${prefix}" can_id="${can_id}" kp="${kp}" kd="${kd}" vel_min="-76.0" vel_max="76.0" effort_min="-12.0" effort_max="12.0" />
   </xacro:macro>
-  <xacro:macro name="AK80-6" params="name prefix can_id Kp Kd">
+  <xacro:macro name="AK80-6" params="name prefix can_id kp kd">
     <xacro:cubemars_ak name="${name}"
                        prefix="${prefix}"
                        can_id="${can_id}"
-                       Kp="${Kp}"
-                       Kd="${Kd}"
+                       kp="${kp}"
+                       kd="${kd}"
                        pos_min="-95.5"
                        pos_max="95.5"
@@ -53,10 +53,10 @@
                        effort_max="18.0" />
   </xacro:macro>
-  <xacro:macro name="AK80-6_V2" params="name prefix can_id Kp Kd">
+  <xacro:macro name="AK80-6_V2" params="name prefix can_id kp kd">
     <xacro:cubemars_ak name="${name}"
                        prefix="${prefix}"
                        can_id="${can_id}"
-                       Kp="${Kp}"
-                       Kd="${Kd}"
+                       kp="${kp}"
+                       kd="${kd}"
                        pos_min="-12.5"
                        pos_max="12.5"
@@ -66,13 +66,13 @@
                        effort_max="12.0" />
   </xacro:macro>
-  <xacro:macro name="AK80-9" params="name prefix can_id Kp Kd">
-    <xacro:cubemars_ak name="${name}" prefix="${prefix}" can_id="${can_id}" Kp="${Kp}" Kd="${Kd}" vel_min="-50.0" vel_max="50.0" effort_min="-18.0" effort_max="18.0"/>
+  <xacro:macro name="AK80-9" params="name prefix can_id kp kd">
+    <xacro:cubemars_ak name="${name}" prefix="${prefix}" can_id="${can_id}" kp="${kp}" kd="${kd}" vel_min="-50.0" vel_max="50.0" effort_min="-18.0" effort_max="18.0"/>
   </xacro:macro>
-  <xacro:macro name="AK80-9_V2" params="name prefix can_id Kp Kd">
+  <xacro:macro name="AK80-9_V2" params="name prefix can_id kp kd">
     <xacro:cubemars_ak name="${name}"
                        prefix="${prefix}"
                        can_id="${can_id}"
-                       Kp="${Kp}"
-                       Kd="${Kd}"
+                       kp="${kp}"
+                       kd="${kd}"
                        pos_min="-12.5"
                        pos_max="12.5"
@@ -80,11 +80,11 @@
                        vel_max="25.64"
                        effort_min="-18.0"
-                       effort_max="18      .0" />
+                       effort_max="18.0" />
   </xacro:macro>
-  <xacro:macro name="AK80-64" params="name prefix can_id Kp Kd">
-    <xacro:cubemars_ak name="${name}" prefix="${prefix}" can_id="${can_id}" Kp="${Kp}" Kd="${Kd}" vel_min="-8.0" vel_max="8.0" effort_min="-144.0" effort_max="144.0"/>
+  <xacro:macro name="AK80-64" params="name prefix can_id kp kd">
+    <xacro:cubemars_ak name="${name}" prefix="${prefix}" can_id="${can_id}" kp="${kp}" kd="${kd}" vel_min="-8.0" vel_max="8.0" effort_min="-144.0" effort_max="144.0"/>
   </xacro:macro>
-  <xacro:macro name="AK80-8" params="name prefix can_id Kp Kd">
-    <xacro:cubemars_ak name="${name}" prefix="${prefix}" can_id="${can_id}" Kp="${Kp}" Kd="${Kd}" vel_min="-37.5" vel_max="37.5" effort_min="-32.0" effort_max="32.0"/>
+  <xacro:macro name="AK80-8" params="name prefix can_id kp kd">
+    <xacro:cubemars_ak name="${name}" prefix="${prefix}" can_id="${can_id}" kp="${kp}" kd="${kd}" vel_min="-37.5" vel_max="37.5" effort_min="-32.0" effort_max="32.0"/>
   </xacro:macro>
 </robot>

Commit message: added parameter to set zero pos on startup

File: ros2_control/cubemars.ros2_control.xacro (robot description, xacro)
@@ -1,5 +1,5 @@
 <?xml version="1.0"?>
 <robot xmlns:xacro="http://www.ros.org/wiki/xacro">
-  <xacro:macro name="cubemars_ak" params="name prefix can_id kp kd vel_min vel_max effort_min effort_max pos_min:=-12.5 pos_max:=12.5 kp_min:=0 kp_max:=500 kd_min:=0 kd_max:=5">
+  <xacro:macro name="cubemars_ak" params="name prefix can_id kp kd vel_min vel_max effort_min effort_max pos_min:=-12.5 pos_max:=12.5 kp_min:=0 kp_max:=500 kd_min:=0 kd_max:=5 invert:=False">
     <joint name="${prefix}${name}">
       <param name="can_id">${can_id}</param>
@@ -10,4 +10,5 @@
       <param name="kd_min">${kd_min}</param>
       <param name="kd_max">${kd_max}</param>
+      <param name="invert">${invert}</param>
       <command_interface name="position">
         <param name="min">${pos_min}</param>
@@ -28,5 +29,5 @@
     </joint>
   </xacro:macro>
-  <xacro:macro name="AK10-9" params="name prefix can_id kp kd">
+  <xacro:macro name="AK10-9" params="name prefix can_id kp kd invert:=False">
     <xacro:cubemars_ak
       name="${name}"
@@ -39,7 +40,8 @@
       effort_min="-65.0"
       effort_max="65.0"
+      invert="${invert}"
     />
   </xacro:macro>
-  <xacro:macro name="AK60-6" params="name prefix can_id kp kd">
+  <xacro:macro name="AK60-6" params="name prefix can_id kp kd invert:=False">
     <xacro:cubemars_ak
       name="${name}"
@@ -52,7 +54,8 @@
       effort_min="-15.0"
       effort_max="15.0"
+      invert="${invert}"
     />
   </xacro:macro>
-  <xacro:macro name="AK70-10" params="name prefix can_id kp kd">
+  <xacro:macro name="AK70-10" params="name prefix can_id kp kd invert:=False">
     <xacro:cubemars_ak
       name="${name}"
@@ -65,7 +68,8 @@
       effort_min="-25.0"
       effort_max="25.0"
+      invert="${invert}"
     />
   </xacro:macro>
-  <xacro:macro name="AK80-5" params="name prefix can_id kp kd">
+  <xacro:macro name="AK80-5" params="name prefix can_id kp kd invert:=False">
     <xacro:cubemars_ak
       name="${name}"
@@ -78,7 +82,8 @@
       effort_min="-12.0"
       effort_max="12.0"
+      invert="${invert}"
     />
   </xacro:macro>
-  <xacro:macro name="AK80-6" params="name prefix can_id kp kd">
+  <xacro:macro name="AK80-6" params="name prefix can_id kp kd invert:=False">
     <xacro:cubemars_ak
       name="${name}"
@@ -93,7 +98,8 @@
       effort_min="-18.0"
       effort_max="18.0"
+      invert="${invert}"
     />
   </xacro:macro>
-  <xacro:macro name="AK80-6_V2" params="name prefix can_id kp kd">
+  <xacro:macro name="AK80-6_V2" params="name prefix can_id kp kd invert:=False">
     <xacro:cubemars_ak
       name="${name}"
@@ -108,7 +114,8 @@
       effort_min="-12.0"
       effort_max="12.0"
+      invert="${invert}"
     />
   </xacro:macro>
-  <xacro:macro name="AK80-9" params="name prefix can_id kp kd">
+  <xacro:macro name="AK80-9" params="name prefix can_id kp kd invert:=False">
     <xacro:cubemars_ak
       name="${name}"
@@ -121,7 +128,8 @@
       effort_min="-18.0"
       effort_max="18.0"
+      invert="${invert}"
     />
   </xacro:macro>
-  <xacro:macro name="AK80-9_V2" params="name prefix can_id kp kd">
+  <xacro:macro name="AK80-9_V2" params="name prefix can_id kp kd invert:=False">
     <xacro:cubemars_ak
       name="${name}"
@@ -136,7 +144,8 @@
       effort_min="-18.0"
       effort_max="18.0"
+      invert="${invert}"
     />
   </xacro:macro>
-  <xacro:macro name="AK80-64" params="name prefix can_id kp kd">
+  <xacro:macro name="AK80-64" params="name prefix can_id kp kd invert:=False">
     <xacro:cubemars_ak name="${name}"
       prefix="${prefix}"
@@ -148,7 +157,8 @@
       effort_min="-144.0"
       effort_max="144.0"
+      invert="${invert}"
     />
   </xacro:macro>
-  <xacro:macro name="AK80-8" params="name prefix can_id kp kd">
+  <xacro:macro name="AK80-8" params="name prefix can_id kp kd invert:=False">
     <xacro:cubemars_ak
       name="${name}"
@@ -161,4 +171,5 @@
       effort_min="-32.0"
       effort_max="32.0"
+      invert="${invert}"
     />
   </xacro:macro>

Commit message: add limits

File: ros2_control/cubemars.ros2_control.xacro (robot description, xacro)
@@ -1,5 +1,9 @@
 <?xml version="1.0"?>
 <robot xmlns:xacro="http://www.ros.org/wiki/xacro">
-  <xacro:macro name="cubemars_ak" params="name prefix can_id kp kd vel_min vel_max effort_min effort_max pos_min:=-12.5 pos_max:=12.5 kp_min:=0 kp_max:=500 kd_min:=0 kd_max:=5 invert:=False">
+  <xacro:macro name="cubemars_ak" params="name prefix can_id kp kd
+                                          vel_min vel_max effort_min effort_max pos_min:=-12.5 pos_max:=12.5
+                                          kp_min:=0 kp_max:=500 kd_min:=0 kd_max:=5
+                                          pos_limit_max:=INF pos_limit_min:=-INF vel_limit_min:=nan vel_limit_max:=nan effort_limit_min:=nan effort_limit_max:=nan
+                                          invert:=False">
     <joint name="${prefix}${name}">
       <param name="can_id">${can_id}</param>
@@ -10,16 +14,22 @@
       <param name="kd_min">${kd_min}</param>
       <param name="kd_max">${kd_max}</param>
+      <param name="pos_min">${pos_min}</param>
+      <param name="pos_max">${pos_max}</param>
+      <param name="vel_min">${vel_min}</param>
+      <param name="vel_max">${vel_max}</param>
+      <param name="effort_min">${effort_min}</param>
+      <param name="effort_max">${effort_max}</param>
       <param name="invert">${invert}</param>
       <command_interface name="position">
-        <param name="min">${pos_min}</param>
-        <param name="max">${pos_max}</param>
+        <param name="min">${pos_limit_min}</param>
+        <param name="max">${pos_limit_max}</param>
       </command_interface>
       <command_interface name="velocity">
-        <param name="min">${vel_min}</param>
-        <param name="max">${vel_max}</param>
+        <param name="min">${vel_limit_min}</param>
+        <param name="max">${vel_limit_max}</param>
       </command_interface>
       <command_interface name="effort">
-        <param name="min">${effort_min}</param>
-        <param name="max">${effort_max}</param>
+        <param name="min">${effort_limit_min}</param>
+        <param name="max">${effort_limit_max}</param>
       </command_interface>
       <state_interface name="position"/>
