Commit message: added soft limits

File: ros2_control/cubemars.ros2_control.xacro (robot description, xacro)
@@ -1,8 +1,16 @@
 <?xml version="1.0"?>
 <robot xmlns:xacro="http://www.ros.org/wiki/xacro">
-  <xacro:macro name="cubemars_ak" params="name prefix can_id kp kd
-                                          vel_min vel_max effort_min effort_max pos_min:=-12.5 pos_max:=12.5
-                                          kp_min:=0 kp_max:=500 kd_min:=0 kd_max:=5
-                                          pos_limit_max:=INF pos_limit_min:=-INF vel_limit_min:=nan vel_limit_max:=nan effort_limit_min:=nan effort_limit_max:=nan
+  <xacro:macro name="cubemars_ak" params="name
+                                          prefix
+                                          can_id
+                                          kp kd
+                                          vel_min vel_max
+                                          effort_min effort_max
+                                          pos_limit_max pos_limit_min
+                                          vel_limit_min vel_limit_max
+                                          effort_limit_min effort_limit_max
+                                          pos_min:=-12.5 pos_max:=12.5
+                                          kp_min:=0 kp_max:=500
+                                          kd_min:=0 kd_max:=5
                                           invert:=False">
     <joint name="${prefix}${name}">
@@ -39,5 +47,15 @@
     </joint>
   </xacro:macro>
-  <xacro:macro name="AK10-9" params="name prefix can_id kp kd invert:=False">
+  <xacro:macro name="AK10-9" params="name
+                                     prefix
+                                     can_id
+                                     kp kd
+                                     pos_limit_min:=-INF
+                                     pos_limit_max:=INF
+                                     vel_limit_min:=-INF
+                                     vel_limit_max:=INF
+                                     effort_limit_min:=-INF
+                                     effort_limit_max:=INF
+                                     invert:=False">
     <xacro:cubemars_ak
       name="${name}"
@@ -50,8 +68,24 @@
       effort_min="-65.0"
       effort_max="65.0"
-      invert="${invert}"
-    />
-  </xacro:macro>
-  <xacro:macro name="AK60-6" params="name prefix can_id kp kd invert:=False">
+      pos_limit_min="${pos_limit_min}"
+      pos_limit_max="${pos_limit_max}"
+      vel_limit_min="${vel_limit_min}"
+      vel_limit_max="${vel_limit_max}"
+      effort_limit_min="${effort_limit_min}"
+      effort_limit_max="${effort_limit_max}"
+      invert="${invert}"
+    />
+  </xacro:macro>
+  <xacro:macro name="AK60-6" params="name
+                                     prefix
+                                     can_id
+                                     kp kd
+                                     pos_limit_min:=-INF
+                                     pos_limit_max:=INF
+                                     vel_limit_min:=-INF
+                                     vel_limit_max:=INF
+                                     effort_limit_min:=-INF
+                                     effort_limit_max:=INF
+                                     invert:=False">
     <xacro:cubemars_ak
       name="${name}"
@@ -64,8 +98,24 @@
       effort_min="-15.0"
       effort_max="15.0"
-      invert="${invert}"
-    />
-  </xacro:macro>
-  <xacro:macro name="AK70-10" params="name prefix can_id kp kd invert:=False">
+      pos_limit_min="${pos_limit_min}"
+      pos_limit_max="${pos_limit_max}"
+      vel_limit_min="${vel_limit_min}"
+      vel_limit_max="${vel_limit_max}"
+      effort_limit_min="${effort_limit_min}"
+      effort_limit_max="${effort_limit_max}"
+      invert="${invert}"
+    />
+  </xacro:macro>
+  <xacro:macro name="AK70-10" params="name
+                                     prefix
+                                     can_id
+                                     kp kd
+                                     pos_limit_min:=-INF
+                                     pos_limit_max:=INF
+                                     vel_limit_min:=-INF
+                                     vel_limit_max:=INF
+                                     effort_limit_min:=-INF
+                                     effort_limit_max:=INF
+                                     invert:=False">
     <xacro:cubemars_ak
       name="${name}"
@@ -78,8 +128,24 @@
       effort_min="-25.0"
       effort_max="25.0"
-      invert="${invert}"
-    />
-  </xacro:macro>
-  <xacro:macro name="AK80-5" params="name prefix can_id kp kd invert:=False">
+      pos_limit_min="${pos_limit_min}"
+      pos_limit_max="${pos_limit_max}"
+      vel_limit_min="${vel_limit_min}"
+      vel_limit_max="${vel_limit_max}"
+      effort_limit_min="${effort_limit_min}"
+      effort_limit_max="${effort_limit_max}"
+      invert="${invert}"
+    />
+  </xacro:macro>
+  <xacro:macro name="AK80-5" params="name
+                                     prefix
+                                     can_id
+                                     kp kd
+                                     pos_limit_min:=-INF
+                                     pos_limit_max:=INF
+                                     vel_limit_min:=-INF
+                                     vel_limit_max:=INF
+                                     effort_limit_min:=-INF
+                                     effort_limit_max:=INF
+                                     invert:=False">
     <xacro:cubemars_ak
       name="${name}"
@@ -92,8 +158,24 @@
       effort_min="-12.0"
       effort_max="12.0"
-      invert="${invert}"
-    />
-  </xacro:macro>
-  <xacro:macro name="AK80-6" params="name prefix can_id kp kd invert:=False">
+      pos_limit_min="${pos_limit_min}"
+      pos_limit_max="${pos_limit_max}"
+      vel_limit_min="${vel_limit_min}"
+      vel_limit_max="${vel_limit_max}"
+      effort_limit_min="${effort_limit_min}"
+      effort_limit_max="${effort_limit_max}"
+      invert="${invert}"
+    />
+  </xacro:macro>
+  <xacro:macro name="AK80-6" params="name
+                                     prefix
+                                     can_id
+                                     kp kd
+                                     pos_limit_min:=-INF
+                                     pos_limit_max:=INF
+                                     vel_limit_min:=-INF
+                                     vel_limit_max:=INF
+                                     effort_limit_min:=-INF
+                                     effort_limit_max:=INF
+                                     invert:=False">
     <xacro:cubemars_ak
       name="${name}"
@@ -108,8 +190,24 @@
       effort_min="-18.0"
       effort_max="18.0"
-      invert="${invert}"
-    />
-  </xacro:macro>
-  <xacro:macro name="AK80-6_V2" params="name prefix can_id kp kd invert:=False">
+      pos_limit_min="${pos_limit_min}"
+      pos_limit_max="${pos_limit_max}"
+      vel_limit_min="${vel_limit_min}"
+      vel_limit_max="${vel_limit_max}"
+      effort_limit_min="${effort_limit_min}"
+      effort_limit_max="${effort_limit_max}"
+      invert="${invert}"
+    />
+  </xacro:macro>
+  <xacro:macro name="AK80-6_V2" params="name
+                                     prefix
+                                     can_id
+                                     kp kd
+                                     pos_limit_min:=-INF
+                                     pos_limit_max:=INF
+                                     vel_limit_min:=-INF
+                                     vel_limit_max:=INF
+                                     effort_limit_min:=-INF
+                                     effort_limit_max:=INF
+                                     invert:=False">
     <xacro:cubemars_ak
       name="${name}"
@@ -124,8 +222,24 @@
       effort_min="-12.0"
       effort_max="12.0"
-      invert="${invert}"
-    />
-  </xacro:macro>
-  <xacro:macro name="AK80-9" params="name prefix can_id kp kd invert:=False">
+      pos_limit_min="${pos_limit_min}"
+      pos_limit_max="${pos_limit_max}"
+      vel_limit_min="${vel_limit_min}"
+      vel_limit_max="${vel_limit_max}"
+      effort_limit_min="${effort_limit_min}"
+      effort_limit_max="${effort_limit_max}"
+      invert="${invert}"
+    />
+  </xacro:macro>
+  <xacro:macro name="AK80-9" params="name
+                                     prefix
+                                     can_id
+                                     kp kd
+                                     pos_limit_min:=-INF
+                                     pos_limit_max:=INF
+                                     vel_limit_min:=-INF
+                                     vel_limit_max:=INF
+                                     effort_limit_min:=-INF
+                                     effort_limit_max:=INF
+                                     invert:=False">
     <xacro:cubemars_ak
       name="${name}"
@@ -138,8 +252,24 @@
       effort_min="-18.0"
       effort_max="18.0"
-      invert="${invert}"
-    />
-  </xacro:macro>
-  <xacro:macro name="AK80-9_V2" params="name prefix can_id kp kd invert:=False">
+      pos_limit_min="${pos_limit_min}"
+      pos_limit_max="${pos_limit_max}"
+      vel_limit_min="${vel_limit_min}"
+      vel_limit_max="${vel_limit_max}"
+      effort_limit_min="${effort_limit_min}"
+      effort_limit_max="${effort_limit_max}"
+      invert="${invert}"
+    />
+  </xacro:macro>
+  <xacro:macro name="AK80-9_V2" params="name
+                                     prefix
+                                     can_id
+                                     kp kd
+                                     pos_limit_min:=-INF
+                                     pos_limit_max:=INF
+                                     vel_limit_min:=-INF
+                                     vel_limit_max:=INF
+                                     effort_limit_min:=-INF
+                                     effort_limit_max:=INF
+                                     invert:=False">
     <xacro:cubemars_ak
       name="${name}"
@@ -154,8 +284,24 @@
       effort_min="-18.0"
       effort_max="18.0"
-      invert="${invert}"
-    />
-  </xacro:macro>
-  <xacro:macro name="AK80-64" params="name prefix can_id kp kd invert:=False">
+      pos_limit_min="${pos_limit_min}"
+      pos_limit_max="${pos_limit_max}"
+      vel_limit_min="${vel_limit_min}"
+      vel_limit_max="${vel_limit_max}"
+      effort_limit_min="${effort_limit_min}"
+      effort_limit_max="${effort_limit_max}"
+      invert="${invert}"
+    />
+  </xacro:macro>
+  <xacro:macro name="AK80-64" params="name
+                                     prefix
+                                     can_id
+                                     kp kd
+                                     pos_limit_min:=-INF
+                                     pos_limit_max:=INF
+                                     vel_limit_min:=-INF
+                                     vel_limit_max:=INF
+                                     effort_limit_min:=-INF
+                                     effort_limit_max:=INF
+                                     invert:=False">
     <xacro:cubemars_ak name="${name}"
       prefix="${prefix}"
@@ -167,8 +313,24 @@
       effort_min="-144.0"
       effort_max="144.0"
-      invert="${invert}"
-    />
-  </xacro:macro>
-  <xacro:macro name="AK80-8" params="name prefix can_id kp kd invert:=False">
+      pos_limit_min="${pos_limit_min}"
+      pos_limit_max="${pos_limit_max}"
+      vel_limit_min="${vel_limit_min}"
+      vel_limit_max="${vel_limit_max}"
+      effort_limit_min="${effort_limit_min}"
+      effort_limit_max="${effort_limit_max}"
+      invert="${invert}"
+    />
+  </xacro:macro>
+  <xacro:macro name="AK80-8" params="name
+                                     prefix
+                                     can_id
+                                     kp kd
+                                     pos_limit_min:=-INF
+                                     pos_limit_max:=INF
+                                     vel_limit_min:=-INF
+                                     vel_limit_max:=INF
+                                     effort_limit_min:=-INF
+                                     effort_limit_max:=INF
+                                     invert:=False">
     <xacro:cubemars_ak
       name="${name}"
@@ -181,4 +343,10 @@
       effort_min="-32.0"
       effort_max="32.0"
+      pos_limit_min="${pos_limit_min}"
+      pos_limit_max="${pos_limit_max}"
+      vel_limit_min="${vel_limit_min}"
+      vel_limit_max="${vel_limit_max}"
+      effort_limit_min="${effort_limit_min}"
+      effort_limit_max="${effort_limit_max}"
       invert="${invert}"
     />
